File: AxxSolder_hardware/AxxSolder.kicad_sch (KiCad schematic)
At the start: 152 parts, among them IC1 TLV76733DRVR, IC2 OPA2387DSGT, IC3 LMR54406DBVR, IC4 STM32G431CBT6, IC5 TPD4E1U06DBVR, IC6 STUSB4500QTR, IC7 MAX16171ATA_VY+T, IC8 LTC4440AHMS8E, IC9 INA281A5QDBVRQ1, J1 USB4110-GF-A, J2 691243110009, J3 TSW-102-07-T-S, J4 61300611821, J5 TSW-102-07-T-S, J6 TSW-102-07-T-S, J7 TSW-108-07-T-S, J8 Conn_01x01_Pin, Q1 STL9P3LLH6, Q2 STL10N3LLH5, Q3 2N7002NXAKR, U2 PEC11J-9215F-S0015, U3 BSC014N04LS

Commit message: set LCSC ID where it's obvious
Parts:
- IC1: LCSC (none) -> C2848334
- IC3: LCSC (none) -> C5219316
- IC4: LCSC (none) -> C529355
- IC5: LCSC (none) -> C124691
- IC6: LCSC (none) -> C2678061
- IC9: LCSC (none) -> C2861018
- J1: LCSC (none) -> C5143397
- J5: LCSC (none) -> C3337281
- J7: LCSC (none) -> C7403228
- L1: LCSC (none) -> C22402289
- Q1: LCSC (none) -> C2969828
- Q2: LCSC (none) -> C2971610
- U3: LCSC (none) -> C2760081
Changed lines of the file:
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@@
       (effects (font (size 1.27 1.27)) (justify left top) hide)
     )
+    (property "LCSC" "C7403228" (at 138.938 77.47 0)
+      (effects (font (size 1.27 1.27)) hide)
+    )
     (pin "6")
     (pin "2")
@@
       (effects (font (size 1.27 1.27)) hide)
     )
+    (property "LCSC" "C2848334" (at 154.94 17.78 0)
+      (effects (font (size 1.27 1.27)) hide)
+    )
     (pin "4")
     (pin "3")
@@
       (effects (font (size 1.27 1.27)) hide)
     )
+    (property "LCSC" "C2971610" (at 16.383 104.394 0)
+      (effects (font (size 1.27 1.27)) hide)
+    )
     (pin "1")
     (pin "4")
@@
       (effects (font (size 1.27 1.27)) hide)
     )
+    (property "LCSC" "C2861018" (at 193.04 110.49 0)
+      (effects (font (size 1.27 1.27)) hide)
+    )
     (pin "1")
     (pin "3")
@@
       (effects (font (size 1.27 1.27)) hide)
     )
+    (property "LCSC" "C5219316" (at 144.145 39.37 0)
+      (effects (font (size 1.27 1.27)) hide)
+    )
     (pin "6")
     (pin "4")
@@
       (effects (font (size 1.27 1.27)) hide)
     )
+    (property "LCSC" "C124691" (at 41.529 70.485 0)
+      (effects (font (size 1.27 1.27)) hide)
+    )
     (pin "1")
     (pin "5")
@@
       (effects (font (size 1.27 1.27)) hide)
     )
+    (property "LCSC" "C529355" (at 266.7 27.94 0)
+      (effects (font (size 1.27 1.27)) hide)
+    )
     (pin "27")
     (pin "24")
@@
       (effects (font (size 1.27 1.27)) hide)
     )
+    (property "LCSC" "C2760081" (at 82.55 166.37 0)
+      (effects (font (size 1.27 1.27)) hide)
+    )
     (pin "1")
     (pin "10")
@@
       (effects (font (size 1.27 1.27)) hide)
     )
+    (property "LCSC" "C3337281" (at 179.578 163.576 0)
+      (effects (font (size 1.27 1.27)) hide)
+    )
     (pin "1")
     (pin "2")
@@
       (effects (font (size 1.27 1.27)) hide)
     )
+    (property "LCSC" "C5143397" (at 16.764 66.04 0)
+      (effects (font (size 1.27 1.27)) hide)
+    )
     (pin "A1")
     (pin "A12")
@@
       (effects (font (size 1.27 1.27)) hide)
     )
+    (property "LCSC" "C2678061" (at 82.55 87.122 0)
+      (effects (font (size 1.27 1.27)) hide)
+    )
     (pin "1")
     (pin "10")
@@
       (effects (font (size 1.27 1.27)) hide)
     )
+    (property "LCSC" "C22402289" (at 171.45 38.735 0)
+      (effects (font (size 1.27 1.27)) hide)
+    )
     (pin "1")
     (pin "2")
@@
       (effects (font (size 1.27 1.27)) hide)
     )
+    (property "LCSC" "C2969828" (at 83.82 64.262 0)
+      (effects (font (size 1.27 1.27)) hide)
+    )

Commit message: add more LCSC IDs
Parts:
- D1: LCSC (none) -> C212291
- D9: LCSC (none) -> C98663
- F1: LCSC (none) -> C206918
- F2: LCSC (none) -> C3156806
- FB1: LCSC (none) -> C88979
- J6: LCSC (none) -> C3337281
- Q3: LCSC (none) -> C551416
Changed lines of the file:
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@@
       (effects (font (size 1.27 1.27)) hide)
     )
+    (property "LCSC" "C3337281" (at 187.706 163.576 0)
+      (effects (font (size 1.27 1.27)) hide)
+    )
     (pin "1")
     (pin "2")
@@
       (effects (font (size 1.27 1.27)) hide)
     )
+    (property "LCSC" "C212291" (at 41.275 24.765 0)
+      (effects (font (size 1.27 1.27)) hide)
+    )
     (pin "1")
     (pin "2")
@@
       (effects (font (size 1.27 1.27)) hide)
     )
+    (property "LCSC" "C206918" (at 182.88 72.39 0)
+      (effects (font (size 1.27 1.27)) hide)
+    )
     (pin "2")
     (pin "1")
@@
       (effects (font (size 1.27 1.27)) hide)
     )
+    (property "LCSC" "C551416" (at 273.685 143.51 0)
+      (effects (font (size 1.27 1.27)) hide)
+    )
     (pin "1")
     (pin "2")
@@
       (effects (font (size 1.27 1.27)) hide)
     )
+    (property "LCSC" "C98663" (at 48.895 160.02 0)
+      (effects (font (size 1.27 1.27)) hide)
+    )
     (pin "1")
     (pin "2")
@@
       (effects (font (size 1.27 1.27)) hide)
     )
+    (property "LCSC" "C3156806" (at 175.26 85.09 0)
+      (effects (font (size 1.27 1.27)) hide)
+    )
     (pin "1")
     (pin "2")
@@
       (effects (font (size 1.27 1.27)) hide)
     )
+    (property "LCSC" "C88979" (at 273.05 100.33 0)
+      (effects (font (size 1.27 1.27)) hide)
+    )

Commit message: add LCSC ID's
Parts:
- C1, C10, C11, C12, C13, C19, C2, C20, C30, C31, C32, C34, C35, C5, C7, C8: LCSC (none) -> C194427
- C37: LCSC (none) -> C136294
- C4, C6: LCSC (none) -> C2839443
- D10: LCSC (none) -> C98663
- D2: LCSC (none) -> C212291
- D3, D4: LCSC (none) -> C5380693
- D5, D6, D7, D8: LCSC (none) -> C916425
- IC7: LCSC (none) -> C3229341
- J2: LCSC (none) -> C5184955
Changed lines of the file:
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@@
       (effects (font (size 1.27 1.27)) hide)
     )
+    (property "LCSC" "C194427" (at 186.69 23.495 0)
+      (effects (font (size 1.27 1.27)) hide)
+    )
     (pin "1")
     (pin "2")
@@
       (effects (font (size 1.27 1.27)) hide)
     )
+    (property "LCSC" "C3229341" (at 46.863 101.219 0)
+      (effects (font (size 1.27 1.27)) hide)
+    )
     (pin "1")
     (pin "2")
@@
       (effects (font (size 1.27 1.27)) hide)
     )
+    (property "LCSC" "C916425" (at 143.51 146.05 0)
+      (effects (font (size 1.27 1.27)) hide)
+    )
     (pin "1")
     (pin "2")
@@
       (effects (font (size 1.27 1.27)) hide)
     )
+    (property "LCSC" "C194427" (at 107.95 173.355 0)
+      (effects (font (size 1.27 1.27)) hide)
+    )
     (pin "1")
     (pin "2")
@@
       (effects (font (size 1.27 1.27)) hide)
     )
+    (property "LCSC" "C194427" (at 71.755 159.385 0)
+      (effects (font (size 1.27 1.27)) hide)
+    )
     (pin "1")
     (pin "2")
@@
       (effects (font (size 1.27 1.27)) hide)
     )
+    (property "LCSC" "C194427" (at 58.42 74.422 0)
+      (effects (font (size 1.27 1.27)) hide)
+    )
     (pin "1")
     (pin "2")
@@
       (effects (font (size 1.27 1.27)) hide)
     )
+    (property "LCSC" "C916425" (at 137.16 125.73 0)
+      (effects (font (size 1.27 1.27)) hide)
+    )
     (pin "1")
     (pin "2")
@@
       (effects (font (size 1.27 1.27)) hide)
     )
+    (property "LCSC" "C5380693" (at 64.77 90.932 0)
+      (effects (font (size 1.27 1.27)) hide)
+    )
     (pin "1")
     (pin "2")
@@
       (effects (font (size 1.27 1.27)) hide)
     )
+    (property "LCSC" "C136294" (at 93.98 173.355 0)
+      (effects (font (size 1.27 1.27)) hide)
+    )
     (pin "1")
     (pin "2")
@@
       (effects (font (size 1.27 1.27)) hide)
     )
+    (property "LCSC" "C916425" (at 89.535 142.24 0)
+      (effects (font (size 1.27 1.27)) hide)
+    )
     (pin "1")
     (pin "2")
@@
       (effects (font (size 1.27 1.27)) hide)
     )
+    (property "LCSC" "C916425" (at 158.75 120.65 0)
+      (effects (font (size 1.27 1.27)) hide)
+    )
     (pin "1")
     (pin "2")
@@
       (effects (font (size 1.27 1.27)) hide)
     )
+    (property "LCSC" "C194427" (at 17.78 173.355 0)
+      (effects (font (size 1.27 1.27)) hide)
+    )
     (pin "1")
     (pin "2")
@@
       (effects (font (size 1.27 1.27)) hide)
     )
+    (property "LCSC" "C98663" (at 89.535 180.34 0)
+      (effects (font (size 1.27 1.27)) hide)
+    )
     (pin "1")
     (pin "2")
@@
       (effects (font (size 1.27 1.27)) hide)
     )
+    (property "LCSC" "C194427" (at 78.105 159.385 0)
+      (effects (font (size 1.27 1.27)) hide)
+    )
     (pin "1")
     (pin "2")
@@
       (effects (font (size 1.27 1.27)) hide)
     )
+    (property "LCSC" "C194427" (at 114.935 74.422 0)
+      (effects (font (size 1.27 1.27)) hide)
+    )
     (pin "1")
     (pin "2")
@@
       (effects (font (size 1.27 1.27)) hide)
     )
+    (property "LCSC" "C194427" (at 104.775 74.422 0)
+      (effects (font (size 1.27 1.27)) hide)
+    )
     (pin "1")
     (pin "2")
@@
       (effects (font (size 1.27 1.27)) hide)
     )
+    (property "LCSC" "C194427" (at 191.77 49.53 0)
+      (effects (font (size 1.27 1.27)) hide)
+    )
     (pin "1")
     (pin "2")
@@
       (effects (font (size 1.27 1.27)) hide)
     )
+    (property "LCSC" "C212291" (at 28.575 42.545 0)
+      (effects (font (size 1.27 1.27)) hide)
+    )
     (pin "1")
     (pin "2")
@@
       (effects (font (size 1.27 1.27)) hide)
     )
+    (property "LCSC" "C194427" (at 100.965 173.355 0)
+      (effects (font (size 1.27 1.27)) hide)
+    )
     (pin "1")
     (pin "2")
@@
       (effects (font (size 1.27 1.27)) hide)
     )
+    (property "LCSC" "C194427" (at 275.59 106.045 0)
+      (effects (font (size 1.27 1.27)) hide)
+    )
     (pin "1")
     (pin "2")
@@
       (effects (font (size 1.27 1.27)) hide)
     )
+    (property "LCSC" "C194427" (at 132.08 44.45 0)
+      (effects (font (size 1.27 1.27)) hide)
+    )
     (pin "1")
     (pin "2")
@@
       (effects (font (size 1.27 1.27)) hide)
     )
+    (property "LCSC" "C194427" (at 198.755 118.11 0)
+      (effects (font (size 1.27 1.27)) hide)
+    )
     (pin "1")
     (pin "2")
@@
       (effects (font (size 1.27 1.27)) hide)
     )
+    (property "LCSC" "C194427" (at 197.485 49.53 0)
+      (effects (font (size 1.27 1.27)) hide)
+    )
     (pin "1")
     (pin "2")
@@
       (effects (font (size 1.27 1.27)) hide)
     )
+    (property "LCSC" "C5380693" (at 165.1 89.535 0)
+      (effects (font (size 1.27 1.27)) hide)
+    )
     (pin "1")
     (pin "2")
@@
       (effects (font (size 1.27 1.27)) hide)
     )
+    (property "LCSC" "C194427" (at 135.255 22.86 0)
+      (effects (font (size 1.27 1.27)) hide)
+    )
     (pin "1")
     (pin "2")
@@
       (effects (font (size 1.27 1.27)) hide)
     )
+    (property "LCSC" "C2839443" (at 67.945 45.085 0)
+      (effects (font (size 1.27 1.27)) hide)
+    )
     (pin "1")
     (pin "2")
@@
       (effects (font (size 1.27 1.27)) hide)
     )
+    (property "LCSC" "C2839443" (at 116.84 45.72 0)
+      (effects (font (size 1.27 1.27)) hide)
+    )
     (pin "1")
     (pin "2")
@@
       (effects (font (size 1.27 1.27)) hide)
     )
+    (property "LCSC" "C5184955" (at 189.23 68.453 0)
+      (effects (font (size 1.27 1.27)) hide)
+    )
     (pin "1")
     (pin "2")
@@
       (effects (font (size 1.27 1.27)) hide)
     )
+    (property "LCSC" "C194427" (at 109.855 74.422 0)
+      (effects (font (size 1.27 1.27)) hide)
+    )

Commit message: add additional ID's
Parts:
- IC2: LCSC (none) -> C5214814
- U2: LCSC (none) -> C32734162
Changed lines of the file:
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@@
       (effects (font (size 1.27 1.27)) hide)
     )
+    (property "LCSC" "C32734162" (at 220.726 133.858 0)
+      (effects (font (size 1.27 1.27)) hide)
+    )
     (pin "A1")
     (pin "B1")
@@
       (effects (font (size 1.27 1.27)) hide)
     )
+    (property "LCSC" "C5214814" (at 69.85 23.495 0)
+      (effects (font (size 1.27 1.27)) hide)
+    )
     (pin "1")
     (pin "2")
@@
       (effects (font (size 1.27 1.27)) hide)
     )
+    (property "LCSC" "C5214814" (at 57.785 42.545 0)
+      (effects (font (size 1.27 1.27)) hide)
+    )
     (pin "1")
     (pin "2")
@@
       (effects (font (size 1.27 1.27)) hide)
     )
+    (property "LCSC" "C5214814" (at 105.41 43.18 0)
+      (effects (font (size 1.27 1.27)) hide)
+    )
